Commit message: 중간저장

File: nuri_humble_desc/urdf/diffbot_description.urdf.xacro (robot description, xacro)
@@ -69,5 +69,5 @@
         <parent link="${prefix}base_link" />
         <child link="${prefix}base_scan" />
-        <origin xyz="0.46 0.225 0.58" rpy="0 0 0" />
+        <origin xyz="0.46 0.225 0.28" rpy="0 0 0" />
     </joint>
   </xacro:macro>
